Commit message: Gazebo Simulation

File: description/robot.urdf.xacro (robot description, xacro)
@@ -2,3 +2,6 @@
 <robot xmlns:xacro="http://www.ros.org/wiki/xacro"  name="robot">
     <xacro:include filename="robot_body.xacro" />
+    <xacro:include filename="gazebo_control.xacro" />
+    <xacro:include filename="lidar.xacro" />
+    <xacro:include filename="camera.xacro" />
 </robot>

File: description/robot_body.xacro (robot description, xacro)
@@ -14,12 +14,14 @@
         <color rgba="0 0 0 1"/>
     </material>
-    <link name="world">
+    <material name="red">
+        <color rgba="1 0 0 1"/>
+    </material>
+    <link name="base_link">
     </link>
-    <joint name="world to base" type="planar">
-        <parent link="world"/>
-        <child link="base_link"/>
-        <origin xyz="0 0 0.1" rpy="0 0 0"/>
+    <joint name="chassis_link" type="fixed">
+        <parent link="base_link"/>
+        <child link="chassis"/>
     </joint>
-    <link name="base_link">
+    <link name="chassis">
         <visual>
             <origin xyz="0 0 0.15" />
@@ -36,17 +38,20 @@
             <material name="orange"/>
         </collision>
-        <xacro:inertial_box mass="0.5" x="0.8" y="0.8" z="0.3">
+        <xacro:inertial_box mass="20.5" x="0.8" y="0.8" z="0.3">
             <origin xyz="0 0 0.15" rpy="0 0 0"/>
         </xacro:inertial_box>
     </link>
+    <gazebo reference="chassis">
+        <material>Gazebo/Red</material>
+    </gazebo>
     <joint name="FL_wheel_link" type="continuous">
-       <parent link="base_link"/>
+       <parent link="chassis"/>
        <child link="FL_wheel"/>
-       <origin xyz="0.2 0.4 0" rpy="-${pi/2} 0 0"/>
+       <origin xyz="0.2 0.45 0" rpy="-${pi/2} 0 0"/>
        <axis xyz="0 0 1"/>
     </joint>
     <link name="FL_wheel">
         <visual>
-            <origin xyz="0 0 0.05" />
+            <origin xyz="0 0 0" />
             <geometry>
                 <cylinder length="0.1" radius="0.1"/>
@@ -55,5 +60,5 @@
         </visual>
         <collision>
-            <origin xyz="0 0 0.05" />
+            <origin xyz="0 0 0" />
             <geometry>
                 <cylinder length="0.1" radius="0.1"/>
@@ -61,16 +66,21 @@
         </collision>
         <xacro:inertial_cylinder mass="0.5" length="0.1" radius="0.1">
-            <origin xyz="0 0 0.05" rpy="0 0 0"/>
+            <origin xyz="0 0 0" rpy="0 0 0"/>
         </xacro:inertial_cylinder>
     </link>
+    <gazebo reference="FL_wheel">
+        <material>Gazebo/White</material>
+        <mu1 value="0.8"/>
+        <mu2 value="0.8"/>
+    </gazebo>
     <joint name="FR_wheel_link" type="continuous">
-        <parent link="base_link"/>
+        <parent link="chassis"/>
         <child link="FR_wheel"/>
-        <origin xyz="0.2 -0.4 0" rpy="${pi/2} 0 0"/>
+        <origin xyz="0.2 -0.45 0" rpy="${pi/2} 0 0"/>
         <axis xyz="0 0 -1"/>
     </joint>
     <link name="FR_wheel">
         <visual>
-            <origin xyz="0 0 0.05"  />
+            <origin xyz="0 0 0"  />
             <geometry>
                 <cylinder length="0.1" radius="0.1"/>
@@ -79,5 +89,5 @@
         </visual>
         <collision>
-            <origin xyz="0 0 0.05" />
+            <origin xyz="0 0 0" />
             <geometry>
                 <cylinder length="0.1" radius="0.1"/>
@@ -85,16 +95,21 @@
         </collision>
         <xacro:inertial_cylinder mass="0.5" length="0.1" radius="0.1">
-            <origin xyz="0 0 0.05" rpy="0 0 0"/>
+            <origin xyz="0 0 0" rpy="0 0 0"/>
         </xacro:inertial_cylinder>
     </link>
+    <gazebo reference="FR_wheel">
+        <material>Gazebo/White</material>
+        <mu1 value="0.8"/>
+        <mu2 value="0.8"/>
+    </gazebo>
     <joint name="BL_wheel_link" type="continuous">
-        <parent link="base_link"/>
+        <parent link="chassis"/>
         <child link="BL_wheel"/>
-        <origin xyz="-0.2 0.4 0" rpy="-${pi/2} 0 0"/>
+        <origin xyz="-0.2 0.45 0" rpy="-${pi/2} 0 0"/>
         <axis xyz="0 0 1"/>
     </joint>
     <link name="BL_wheel">
         <visual>
-            <origin xyz="0 0 0.05" />
+            <origin xyz="0 0 0" />
             <geometry>
                 <cylinder length="0.1" radius="0.1"/>
@@ -103,5 +118,5 @@
         </visual>
         <collision>
-            <origin xyz="0 0 0.05" />
+            <origin xyz="0 0 0" />
             <geometry>
                 <cylinder length="0.1" radius="0.1"/>
@@ -109,16 +124,21 @@
         </collision>
         <xacro:inertial_cylinder mass="0.5" length="0.1" radius="0.1">
-            <origin xyz="0 0 0.05" rpy="0 0 0"/>
+            <origin xyz="0 0 0" rpy="0 0 0"/>
         </xacro:inertial_cylinder>
     </link>
+    <gazebo reference="BL_wheel">
+        <material>Gazebo/White</material>
+        <mu1 value="0.8"/>
+        <mu2 value="0.8"/>
+    </gazebo>
     <joint name="BR_wheel_link" type="continuous">
-        <parent link="base_link"/>
+        <parent link="chassis"/>
         <child link="BR_wheel"/>
-        <origin xyz="-0.2 -0.4 0" rpy="${pi/2} 0 0"/>
+        <origin xyz="-0.2 -0.45 0" rpy="${pi/2} 0 0"/>
         <axis xyz="0 0 -1"/>
     </joint>
     <link name="BR_wheel">
         <visual>
-            <origin xyz="0 0 0.05" />
+            <origin xyz="0 0 0" />
             <geometry>
                 <cylinder length="0.1" radius="0.1"/>
@@ -127,5 +147,5 @@
         </visual>
         <collision>
-            <origin xyz="0 0 0.05" />
+            <origin xyz="0 0 0" />
             <geometry>
                 <cylinder length="0.1" radius="0.1"/>
@@ -133,6 +153,11 @@
         </collision>
         <xacro:inertial_cylinder mass="0.5" length="0.1" radius="0.1">
-            <origin xyz="0 0 0.05" rpy="0 0 0"/>
+            <origin xyz="0 0 0" rpy="0 0 0"/>
         </xacro:inertial_cylinder>
     </link>
+    <gazebo reference="BR_wheel">
+        <material>Gazebo/White</material>
+        <mu1 value="0.8"/>
+        <mu2 value="0.8"/>
+    </gazebo>
 </robot>
